Commit message: [cartographer_ros] Drop the leading slash in turtlebot.urdf frame_ids. (#19)
In tf2, frame_ids should not start with a slash:
http://wiki.ros.org/tf2/Migration

Original commit:
googlecartographer/cartographer_ros@df1b66935b881d77a9fe4d708cc58f0bc3d6b602

File: cartographer_ros/cartographer_ros/urdf/turtlebot.urdf (robot description, URDF)
Before this commit: robot cartographer_ros, 2 links, 1 joints
Links:
- removed link /base_link
- removed link /horizontal_laser_link
- added link base_link; visual box size=0.03 0.4 0.8
- added link horizontal_laser_link; visual cylinder length=0.09 radius=0.03
Joints:
- joint horizontal_laser_link_joint: child /horizontal_laser_link -> horizontal_laser_link; parent /base_link -> base_link

Commit message: [cartographer_ros] Add support for 2D SLAM with a depth camera. (#54)
This changes the URDF and timeout for the TurtleBot configuration,
and adds a Dockerfile with everything that is needed to run 2D SLAM
with a depth camera. Verified to work on a TurtleBot 2 with an
ASUS Xtion.

And tiny style fixes.

Original commit:
googlecartographer/cartographer_ros@0e26c9feac33cc8a86159aeb2ac270d312a9670c

File: cartographer_ros/cartographer_ros/urdf/turtlebot.urdf (robot description, URDF)
Before this commit: robot cartographer_ros, 2 links, 1 joints
Links:
- added link base_footprint
- added link camera_link
Joints:
- added joint base_link_base_footprint_joint: type fixed, parent base_footprint, child base_link, origin xyz=0. 0. 0.
- added joint camera_link_joint: type fixed, parent base_link, child camera_link, origin xyz=0.15 0. 0.6
