Commit message: [cartographer_ros] Add code to allow offline processing of 2D Cartographer bags. (#1)
* Add code to allow offline processing of 2D Cartographer bags.

Fixes waiting for transforms to be published, adds support for multi-echo
laser scans, sets default values for the submap topic and query for the
RViz plugin.

Original commit:
googlecartographer/cartographer_ros@961afb68175e64a57d7acbb809da9053d0586b33

File: cartographer_ros/cartographer_ros/urdf/backpack_2d.urdf (robot description, URDF)
Before this commit: robot cartographer_ros, 4 links, 3 joints
Links:
- removed link /base_footprint
- removed link /horizontal_laser_link
- removed link /imu_link
- removed link /vertical_laser_link
- added link base_link; visual box size=0.03 0.4 0.8
- added link horizontal_laser_link; visual cylinder length=0.09 radius=0.03
- added link imu_link; visual box size=0.055 0.055 0.02
- added link vertical_laser_link; visual cylinder length=0.09 radius=0.03
Joints:
- removed joint base_link_joint
- added joint imu_link_joint: type fixed, parent base_link, child imu_link, origin xyz=0 0 0 rpy=0 0 3.1416
- joint horizontal_laser_link_joint: child /horizontal_laser_link -> horizontal_laser_link; parent /imu_link -> base_link
- joint vertical_laser_link_joint: child /vertical_laser_link -> vertical_laser_link; parent /imu_link -> base_link

Commit message: [cartographer_ros] Fix draw ordering issue of the RViz visualization. (#5)
Instead of drawing into a offscreen texture and blitting the
result as an overlay (which shows up on top of everything else)
we directly draw to the RViz scene. To get proper X-rays one
should use a 0.5 gray background for now.

Also fixes the configuration to enable 3D mapping from a bag.

Original commit:
googlecartographer/cartographer_ros@5497e9c343b247d1e07e79a80cb75b3dcbe44bf3

File: cartographer_ros/cartographer_ros/urdf/backpack_2d.urdf (robot description, URDF)
Before this commit: robot cartographer_ros, 4 links, 3 joints
Links:
- link base_link: geometry 
- link imu_link: geometry visual box size=0.06 0.04 0.02

File: cartographer_ros/cartographer_ros/urdf/backpack_3d.urdf (robot description, URDF)
Before this commit: robot cartographer_ros, 4 links, 3 joints
Links:
- removed link /base_link
- removed link /horizontal_vlp16_link
- removed link /imu_link
- removed link /vertical_vlp16_link
- added link base_link
- added link horizontal_vlp16_link; visual cylinder length=0.07 radius=0.05
- added link imu_link; visual box size=0.06 0.04 0.02
- added link vertical_vlp16_link; visual cylinder length=0.07 radius=0.05
Joints:
- removed joint base_link_joint
- added joint imu_link_joint: type fixed, parent base_link, child imu_link, origin xyz=0 0 0 rpy=3.1416 0 0
- joint horizontal_vlp16_link_joint: child /horizontal_vlp16_link -> horizontal_vlp16_link; parent /base_link -> base_link
- joint vertical_vlp16_link_joint: child /vertical_vlp16_link -> vertical_vlp16_link; parent /base_link -> base_link

Commit message: [cartographer_ros] Improve the 2D backpack URDF. (#96) Original commit: googlecartographer/cartographer_ros@61183d5dbc6df6c49f0c84d2a7a27cbb504c2102

File: cartographer_ros/cartographer_ros/urdf/backpack_2d.urdf (robot description, URDF)
Before this commit: robot cartographer_backpack_2d, 4 links, 3 joints
Links:
- link horizontal_laser_link: geometry visual cylinder length=0.05 radius=0.03
- link vertical_laser_link: geometry visual cylinder length=0.05 radius=0.03
Joints:
- joint horizontal_laser_link_joint: origin xyz=0.1251 0.0937 0.05262 -> xyz=0.1007 0 0.0558
- joint imu_link_joint: origin xyz=0 0 0 rpy=0 0 3.1416 -> xyz=0 0 0 rpy=0 0 3.141593
- joint vertical_laser_link_joint: origin xyz=0.1251 0.0937 0.17772 rpy=0.0 -1.57 3.14 -> xyz=0.1007 0 0.1814 rpy=0 -1.570796 3.141593

Commit message: [cartographer_ros] Fix the IMU orientation in the 2D backpack URDF. (#103) Original commit: googlecartographer/cartographer_ros@0e8d219eef6c7a823d77e6deabf1d89e261e3b77

File: cartographer_ros/cartographer_ros/urdf/backpack_2d.urdf (robot description, URDF)
Before this commit: robot cartographer_backpack_2d, 4 links, 3 joints
Joints:
- joint imu_link_joint: origin xyz=0 0 0 rpy=0 0 3.141593 -> xyz=0 0 0
